File: power.kicad_sch (KiCad schematic)
At the start: 12 parts, among them U2 MP2696A

Commit message: Adding switch to power
Parts:
- C1, C3: value (none) -> 10u 16V; footprint (none) -> Capacitor_SMD:C_0805_2012Metric_Pad1.18x1.45mm_HandSolder
- C2: value (none) -> 1u 16V; footprint (none) -> Capacitor_SMD:C_0805_2012Metric_Pad1.18x1.45mm_HandSolder
- C4: value (none) -> 2.2u 6.3V; footprint (none) -> Capacitor_SMD:C_0805_2012Metric_Pad1.18x1.45mm_HandSolder
- C5: value (none) -> 470n 10V; footprint (none) -> Capacitor_SMD:C_0805_2012Metric_Pad1.18x1.45mm_HandSolder
- C6: value (none) -> 22u 10V; footprint (none) -> Capacitor_SMD:C_0805_2012Metric_Pad1.18x1.45mm_HandSolder
- L1: value (none) -> 1uH; footprint (none) -> Inductor_SMD:L_12x12mm_H4.5mm
- R1: value (none) -> 10m; footprint (none) -> Resistor_SMD:R_0805_2012Metric_Pad1.20x1.40mm_HandSolder
- R2, R3: value (none) -> 10k; footprint (none) -> Resistor_SMD:R_0805_2012Metric_Pad1.20x1.40mm_HandSolder
- U2: footprint (none) -> Library:QFN-21
Changed lines of the file:
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@@
     (property "Reference" "U2" (id 0) (at 116.205 68.9862 0))
     (property "Value" "MP2696A" (id 1) (at 116.205 71.5262 0))
-    (property "Footprint" "" (id 2) (at 75.565 69.85 0)
+    (property "Footprint" "Library:QFN-21" (id 2) (at 75.565 69.85 0)
       (effects (font (size 1.27 1.27)) hide)
     )
@@
       (effects (font (size 1.27 1.27)) (justify left))
     )
-    (property "Value" "" (id 1) (at 144.78 71.12 0)
+    (property "Value" "470n 10V" (id 1) (at 144.78 71.12 0)
       (effects (font (size 1.27 1.27)) (justify left))
     )
-    (property "Footprint" "" (id 2) (at 144.4752 72.39 0)
+    (property "Footprint" "Capacitor_SMD:C_0805_2012Metric_Pad1.18x1.45mm_HandSolder" (id 2) (at 144.4752 72.39 0)
       (effects (font (size 1.27 1.27)) hide)
     )
@@
       (effects (font (size 1.27 1.27)) (justify left))
     )
-    (property "Value" "" (id 1) (at 181.61 85.0899 0)
+    (property "Value" "22u 10V" (id 1) (at 181.61 85.0899 0)
       (effects (font (size 1.27 1.27)) (justify left))
     )
-    (property "Footprint" "" (id 2) (at 178.7652 87.63 0)
+    (property "Footprint" "Capacitor_SMD:C_0805_2012Metric_Pad1.18x1.45mm_HandSolder" (id 2) (at 178.7652 87.63 0)
       (effects (font (size 1.27 1.27)) hide)
     )
@@
     (in_bom yes) (on_board yes)
     (property "Reference" "L1" (id 0) (at 148.59 77.47 90))
-    (property "Value" "" (id 1) (at 153.67 77.47 90))
-    (property "Footprint" "" (id 2) (at 152.4 76.2 0)
+    (property "Value" "1uH" (id 1) (at 153.67 77.47 90))
+    (property "Footprint" "Inductor_SMD:L_12x12mm_H4.5mm" (id 2) (at 152.4 76.2 0)
       (effects (font (size 1.27 1.27)) hide)
     )
@@
     (in_bom yes) (on_board yes) (fields_autoplaced)
     (property "Reference" "C1" (id 0) (at 86.36 58.42 90))
-    (property "Value" "" (id 1) (at 86.36 60.96 90))
-    (property "Footprint" "" (id 2) (at 90.17 65.0748 0)
+    (property "Value" "10u 16V" (id 1) (at 86.36 60.96 90))
+    (property "Footprint" "Capacitor_SMD:C_0805_2012Metric_Pad1.18x1.45mm_HandSolder" (id 2) (at 90.17 65.0748 0)
       (effects (font (size 1.27 1.27)) hide)
     )
@@
       (effects (font (size 1.27 1.27)) (justify left))
     )
-    (property "Value" "" (id 1) (at 93.98 78.7399 0)
+    (property "Value" "1u 16V" (id 1) (at 93.98 78.7399 0)
       (effects (font (size 1.27 1.27)) (justify left))
     )
-    (property "Footprint" "" (id 2) (at 91.1352 81.28 0)
+    (property "Footprint" "Capacitor_SMD:C_0805_2012Metric_Pad1.18x1.45mm_HandSolder" (id 2) (at 91.1352 81.28 0)
       (effects (font (size 1.27 1.27)) hide)
     )
@@
       (effects (font (size 1.27 1.27)) (justify left))
     )
-    (property "Value" "" (id 1) (at 140.97 46.9899 0)
+    (property "Value" "10u 16V" (id 1) (at 140.97 46.9899 0)
       (effects (font (size 1.27 1.27)) (justify left))
     )
-    (property "Footprint" "" (id 2) (at 138.1252 49.53 0)
+    (property "Footprint" "Capacitor_SMD:C_0805_2012Metric_Pad1.18x1.45mm_HandSolder" (id 2) (at 138.1252 49.53 0)
       (effects (font (size 1.27 1.27)) hide)
     )
@@
       (effects (font (size 1.27 1.27)) (justify left))
     )
-    (property "Value" "" (id 1) (at 193.04 96.52 90)
+    (property "Value" "10k" (id 1) (at 193.04 96.52 90)
       (effects (font (size 1.27 1.27)) (justify left))
     )
-    (property "Footprint" "" (id 2) (at 191.77 98.298 90)
+    (property "Footprint" "Resistor_SMD:R_0805_2012Metric_Pad1.20x1.40mm_HandSolder" (id 2) (at 191.77 98.298 90)
       (effects (font (size 1.27 1.27)) hide)
     )
@@
       (effects (font (size 1.27 1.27)) (justify left))
     )
-    (property "Value" "" (id 1) (at 180.34 96.52 90)
+    (property "Value" "10k" (id 1) (at 180.34 96.52 90)
       (effects (font (size 1.27 1.27)) (justify left))
     )
-    (property "Footprint" "" (id 2) (at 179.07 98.298 90)
+    (property "Footprint" "Resistor_SMD:R_0805_2012Metric_Pad1.20x1.40mm_HandSolder" (id 2) (at 179.07 98.298 90)
       (effects (font (size 1.27 1.27)) hide)
     )
@@
     (in_bom yes) (on_board yes)
     (property "Reference" "R1" (id 0) (at 163.83 73.66 90))
-    (property "Value" "" (id 1) (at 163.83 76.2 90))
-    (property "Footprint" "" (id 2) (at 163.83 77.978 90)
+    (property "Value" "10m" (id 1) (at 163.83 76.2 90))
+    (property "Footprint" "Resistor_SMD:R_0805_2012Metric_Pad1.20x1.40mm_HandSolder" (id 2) (at 163.83 77.978 90)
       (effects (font (size 1.27 1.27)) hide)
     )
@@
       (effects (font (size 1.27 1.27)) (justify left))
     )
-    (property "Value" "" (id 1) (at 142.24 110.4899 0)
+    (property "Value" "2.2u 6.3V" (id 1) (at 142.24 110.4899 0)
       (effects (font (size 1.27 1.27)) (justify left))
     )
-    (property "Footprint" "" (id 2) (at 139.3952 113.03 0)
+    (property "Footprint" "Capacitor_SMD:C_0805_2012Metric_Pad1.18x1.45mm_HandSolder" (id 2) (at 139.3952 113.03 0)
       (effects (font (size 1.27 1.27)) hide)
     )
